File: Dayspring/Dayspring.kicad_pcb (KiCad board)
At the start: 2 copper layers, 310 x 11 mm, 55 parts, among them J1 Conn_01x02, J2 Conn_01x02

Commit message: Production Version LED and 3030 Mounts
Parts:
- removed the REF** at (33.1, 38.1)
- removed the REF** at (58.1, 38.1)
- removed the REF** at (108.1, 38.1)
- removed the REF** at (322.1, 32.1)
- removed the REF** at (134.1, 27.1)
- removed the REF** at (160.1, 38.1)
- removed the REF** at (134.1, 38.1)
- removed the REF** at (83.1, 27.1)
- removed the REF** at (83.1, 38.1)
- removed the REF** at (237.1, 38.1)
- removed the REF** at (108.1, 27.1)
- removed the REF** at (186.1, 38.1)
- removed the REF** at (211.1, 38.1)
- removed the REF** at (58.1, 27.1)
- removed the REF** at (263.1, 38.1)
- removed the REF** at (160.1, 27.1)
- removed the REF** at (237.1, 27.1)
- removed the REF** at (186.1, 27.1)
- removed the REF** at (33.1, 27.1)
- removed the REF** at (211.1, 27.1)
- removed the REF** at (13.1, 32.6)
- removed the REF** at (263.1, 27.1)
- added G***: LOGO, LOGO, B.Cu at (220.5, 32.5)
- added J2: Conn_01x02, Connector_PinSocket_2.54mm:PinSocket_1x02_P2.54mm_Horizontal, B.Cu at (24.8, 34.0)
- added J4: Conn_01x02, Connector_PinSocket_2.54mm:PinSocket_1x02_P2.54mm_Horizontal, B.Cu at (313.2, 31.0)
- added REF**: Tab, kikit:Tab, F.Cu at (58.0, 27.1)
- added REF**: Tab, kikit:Tab, F.Cu at (280.0, 37.9)
- added REF**: Tab, kikit:Tab, F.Cu at (280.0, 27.1)
- added REF**: Tab, kikit:Tab, F.Cu at (58.0, 37.9)
- moved R4 39.7 mm to (297.8, 32.5), turned to 90 degrees
- moved R1 24.1 mm to (40.5, 32.5), turned to 90 degrees
- moved J1 19.4 mm to (45.5, 33.8)
- moved J3 17.1 mm to (293.0, 31.2)
- moved R6 15.9 mm to (191.0, 32.5), turned to 90 degrees
- moved G*** 12.4 mm to (31.0, 32.5)
- moved D21 10.9 mm to (317.0, 32.5)
- moved G*** 10.6 mm to (307.0, 32.5), turned to 0 degrees
- moved D18 9.91 mm to (302.2, 32.5)
- moved R5 9.16 mm to (87.2, 32.5), turned to 90 degrees
- moved D1 9.09 mm to (21.0, 32.5)
- moved D15 8.91 mm to (287.4, 32.5)
- moved D4 8.09 mm to (35.8, 32.5)
- moved D12 7.91 mm to (272.6, 32.5)
- moved D7 7.09 mm to (50.6, 32.5)
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- renumbered D4 to D10, D10 to D11, D16 to D12, D5 to D13, D11 to D14, D17 to D15, D6 to D16, D12 to D17, D7 to D2, D13 to D3, D2 to D4, D8 to D5, D14 to D6, D3 to D7, D9 to D8, D15 to D9, J2 to J1, J1 to J3, R5 to R2, R6 to R4, R2 to R5, R4 to R6
Connections:
- D10 pad 1: Net-(D4-Pad1) -> Net-(D10-Pad1)
- D10 pad 2: Net-(D4-Pad2) -> Net-(D10-Pad2)
- D11 pad 1: Net-(D10-Pad1) -> Net-(D11-Pad1)
- D12 pad 2: Net-(D16-Pad2) -> Net-(D12-Pad2)
- D13 pad 1: Net-(D5-Pad1) (its old number) -> Net-(D13-Pad1)
- D13 pad 2: Net-(D5-Pad2) -> Net-(D10-Pad1)
- D14 pad 1: Net-(D11-Pad1) -> Net-(D14-Pad1)
- D14 pad 2: Net-(D11-Pad2) (its old number) -> Net-(D11-Pad1)
- D15 pad 1: Net-(D17-Pad1) (its old number) -> Net-(D15-Pad1)
- D16 pad 2: Net-(D5-Pad1) (its old number) -> Net-(D16-Pad2)
- D17 pad 2: Net-(D11-Pad1) -> Net-(D17-Pad2)
- D18 pad 2: Net-(D17-Pad1) (its old number) -> Net-(D18-Pad2)
- D4 pad 1: Net-(D2-Pad1) (its old number) -> Net-(D4-Pad1)
- D7 pad 1: Net-(D3-Pad1) (its old number) -> Net-(D10-Pad2)
- D7 pad 2: Net-(D2-Pad1) (its old number) -> Net-(D7-Pad2)
- D9 pad 1: Net-(D15-Pad1) -> Net-(D12-Pad2)
- R1 pad 1: Net-(D4-Pad2) -> Net-(D7-Pad2)
- R1 pad 2: Net-(D3-Pad1) (its old number) -> Net-(D4-Pad1)
- R4 pad 1: Net-(D16-Pad2) -> Net-(D18-Pad2)
- R5 pad 1: Net-(D5-Pad2) -> Net-(D16-Pad2)
- R5 pad 2: Net-(D4-Pad1) -> Net-(D13-Pad1)
- R6 pad 1: Net-(D11-Pad2) (its old number) -> Net-(D17-Pad2)
- R6 pad 2: Net-(D10-Pad1) -> Net-(D14-Pad1)
Routing:
- net Net-(D10-Pad2): track 0.00 -> 18.0 mm
- net Net-(D17-Pad1) (its old number): track 17.7 -> 0.00 mm
- net Net-(D2-Pad1) (its old number): track 17.7 -> 0.00 mm
- net Net-(D12-Pad2): track 0.00 -> 15.7 mm
- net Net-(D5-Pad1) (its old number): track 14.7 -> 0.00 mm
- net Net-(D7-Pad2): track 0.00 -> 12.9 mm
- net Net-(D17-Pad2): track 0.00 -> 8.78 mm
- net Net-(D10-Pad1): track 7.23 -> 15.7 mm
- net Net-(D14-Pad1): track 0.00 -> 8.18 mm
- net Net-(D13-Pad1): track 0.00 -> 8.03 mm
- net Net-(D5-Pad2): track 7.24 -> 0.00 mm
- net Net-(D3-Pad1) (its old number): track 7.13 -> 0.00 mm
- net Net-(D4-Pad2): track 6.94 -> 0.00 mm
- net Net-(D11-Pad2) (its old number): track 6.84 -> 0.00 mm
- net Net-(D15-Pad1): track 7.43 -> 13.6 mm
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Other:
- outline, holes or cut-outs redrawn
- board text added: "24V GND"
- board text added: "Daylight on a stick by Blamm Dayspring by Vector 3D V2.0"
- board text added: "GND 24V"
- board text added: "JLCJLCJLCJLC"
- board text removed: "+24V GND"
- board text removed: "- +"
- board text removed: "Daylight on a stick by Blamm Dayspring by Vector 3D V1.0"
- board text removed: "GND +24V"
- board text removed: "JLCJLCJLC"
