File: Dayspring/Dayspring.kicad_sch (KiCad schematic)
At the start: 31 parts, among them J1 Conn_01x02, J2 Conn_01x02

Commit message: Production Version LED and 3030 Mounts
Parts:
- added J2, J4: Conn_01x02, Connector_PinSocket_2.54mm:PinSocket_1x02_P2.54mm_Horizontal, symbol Connector_Generic:Conn_01x02
- J1: renamed from J2; LCSC (none) -> C157931; now in the parts list
- J3: renamed from J1; LCSC (none) -> C157931; now in the parts list
- renumbered D4 to D10, D10 to D11, D16 to D12, D5 to D13, D11 to D14, D17 to D15, D6 to D16, D12 to D17, D7 to D2, D13 to D3, D2 to D4, D8 to D5, D14 to D6, D3 to D7, D9 to D8, D15 to D9, R5 to R2, R6 to R4, R2 to R5, R4 to R6
Connections:
- net +24V: now also J2.2 (Pin_2), J4.1 (Pin_1)
- net GND: now also J2.1 (Pin_1), J4.2 (Pin_2)
- net at D18.2 (A): now also R4.1; no longer D15.1 (K)
- net at D12.2 (A): now also D9.1 (K); no longer R4.1
- net at D7.1 (K): now also D10.2 (A); no longer R1.2
- net at D7.2 (A): now also R1.1; no longer D4.1 (K)
- net at D14.1 (K): now also R6.2; no longer D17.2 (A)
- net at D14.2 (A): now also D11.1 (K); no longer R6.1
- net at D16.2 (A): now also R5.1; no longer D13.1 (K)
- net at R4.2: now also D15.1 (K); no longer D9.1 (K)
- net at D10.1 (K): now also D13.2 (A); no longer R5.2
- new net: D4.1 (K), R1.2
- new net: D17.2 (A), R6.1
- new net: D13.1 (K), R5.2
Other:
- moved on the sheet: D12, D13, D14, D15, D7, R1, R4, R5, R6
