File: Dayspring_Mini/Dayspring_Mini.kicad_pcb (KiCad board)
At the start: 2 copper layers, 170 x 11 mm, 24 parts, among them J1 Conn_01x02, J2 Conn_01x02

Commit message: Production Version LED and 3030 Mounts
Parts:
- removed the G*** at (18.0, 33.0)
- removed the G*** at (178.0, 33.0)
- added G***: LOGO, Daylight:RR_Logo_9mm_F-Silk, F.Cu at (206.5, 33.0)
- added G***: LOGO, Daylight:RR_Logo_9mm_F-Silk, F.Cu at (30.8, 33.0)
- added G***: LOGO, LOGO, B.Cu at (157.8, 33.0)
- added J2: Conn_01x02, Connector_PinSocket_2.54mm:PinSocket_1x02_P2.54mm_Horizontal, B.Cu at (24.2, 34.3)
- added J4: Conn_01x02, Connector_PinSocket_2.54mm:PinSocket_1x02_P2.54mm_Horizontal, B.Cu at (212.8, 31.8)
- added REF**: Tab, kikit:Tab, F.Cu at (57.8, 38.4)
- added REF**: Tab, kikit:Tab, F.Cu at (179.5, 27.6)
- added REF**: Tab, kikit:Tab, F.Cu at (179.5, 38.4)
- added REF**: Tab, kikit:Tab, F.Cu at (57.8, 27.6)
- moved R4 55.5 mm to (196.5, 33.0), turned to 90 degrees
- moved D14 50.0 mm to (216.5, 33.0)
- moved D12 45.5 mm to (201.4, 33.0)
- moved D10 40.9 mm to (186.3, 33.0)
- moved D8 36.4 mm to (171.3, 33.0)
- moved D6 31.8 mm to (156.2, 33.0)
- moved R2 29.0 mm to (148.5, 33.0)
- moved H2 28.8 mm to (179.5, 33.0)
- moved D4 27.3 mm to (141.1, 33.0)
- moved D2 22.8 mm to (126.0, 33.0)
- moved J3 22.5 mm to (192.5, 31.8)
- moved R3 21.8 mm to (88.0, 33.0)
- moved J1 18.5 mm to (44.5, 34.2)
- moved D13 18.2 mm to (111.0, 33.0)
- moved R1 15.5 mm to (40.2, 33.0), turned to 90 degrees
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- renumbered D12 to D10, D6 to D11, D13 to D12, D7 to D13, D8 to D2, D2 to D3, D9 to D4, D3 to D5, D10 to D6, D4 to D7, D11 to D8, D5 to D9, J2 to J3, R3 to R2, R2 to R3
Connections:
- D10 pad 1: Net-(D12-Pad1) (its old number) -> Net-(D10-Pad1)
- D10 pad 2: Net-(D12-Pad2) -> Net-(D10-Pad2)
- D11 pad 2: Net-(D5-Pad1) -> Net-(D11-Pad2)
- D12 pad 2: Net-(D12-Pad1) (its old number) -> Net-(D12-Pad2)
- D3 pad 1: Net-(D2-Pad1) (its old number) -> Net-(D3-Pad1)
- D5 pad 1: Net-(D3-Pad1) -> Net-(D5-Pad1)
- D5 pad 2: Net-(D2-Pad1) (its old number) -> Net-(D5-Pad2)
- D7 pad 1: Net-(D4-Pad1) (its old number) -> Net-(D7-Pad1)
- D7 pad 2: Net-(D4-Pad2) -> Net-(D5-Pad1)
- D8 pad 1: Net-(D11-Pad1) (its old number) -> Net-(D10-Pad2)
- D9 pad 1: Net-(D5-Pad1) -> Net-(D9-Pad1)
- D9 pad 2: Net-(D5-Pad2) -> Net-(D7-Pad1)
- R1 pad 1: Net-(D4-Pad2) -> Net-(D5-Pad2)
- R3 pad 1: Net-(D5-Pad2) -> Net-(D11-Pad2)
- R3 pad 2: Net-(D4-Pad1) (its old number) -> Net-(D9-Pad1)
- R4 pad 2: Net-(D11-Pad1) (its old number) -> Net-(D10-Pad1)
Routing:
- net Net-(D10-Pad2): track 0.00 -> 19.2 mm
- net Net-(D7-Pad1): track 0.00 -> 16.0 mm
- net Net-(D12-Pad1) (its old number): track 14.9 -> 0.00 mm
- net Net-(D2-Pad1) (its old number): track 14.6 -> 0.00 mm
- net Net-(D10-Pad1): track 0.00 -> 13.8 mm
- net Net-(D11-Pad2): track 0.00 -> 9.06 mm
- net Net-(D9-Pad1): track 0.00 -> 8.17 mm
- net Net-(D12-Pad1): track 11.5 -> 19.3 mm
- net Net-(D1-Pad1): track 11.5 -> 19.2 mm
- net Net-(D5-Pad1): track 11.5 -> 18.9 mm
- net Net-(D5-Pad2): track 6.56 -> 13.0 mm
- net Net-(D11-Pad1) (its old number): track 6.24 -> 0.00 mm
- net Net-(D4-Pad1) (its old number): track 6.13 -> 0.00 mm
- net Net-(D4-Pad2): track 5.51 -> 0.00 mm
- net GND: track 5.12 -> 0.00 mm, vias 28 -> 39
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Other:
- board size 170 x 11 mm -> 210 x 11 mm
- board text added: "Daylight on a stick by Blamm Dayspring Mini by Vector 3D V2.0"
- board text added: "JLCJLCJLCJLC"
- board text removed: "Daylight on a stick by Blamm Daybreak Mini by Vector 3D V2.2"
- board text removed: "JLCJLCJLC"
