File: Dayspring_Mini/Dayspring_Mini.kicad_sch (KiCad schematic)
At the start: 22 parts, among them J1 Conn_01x02, J2 Conn_01x02

Commit message: Production Version LED and 3030 Mounts
Parts:
- added J2, J4: Conn_01x02, Connector_PinSocket_2.54mm:PinSocket_1x02_P2.54mm_Horizontal, symbol Connector_Generic:Conn_01x02
- H1, H2: footprint (none) -> MountingHole:MountingHole_3.2mm_M3_Pad_Via
- J1: LCSC (none) -> C157931; now in the parts list
- J3: renamed from J2; LCSC (none) -> C157931; now in the parts list
- renumbered D12 to D10, D6 to D11, D13 to D12, D7 to D13, D8 to D2, D2 to D3, D9 to D4, D3 to D5, D10 to D6, D4 to D7, D11 to D8, D5 to D9, R3 to R2, R2 to R3
Connections:
- net +24V: now also J2.2 (Pin_2), J4.1 (Pin_1)
- net GND: now also J2.1 (Pin_1), J4.2 (Pin_2)
- net at D5.1 (K): now also D7.2 (A); no longer R1.2
- net at D5.2 (A): now also R1.1; no longer D3.1 (K)
- net at D10.1 (K): now also R4.2; no longer D12.2 (A)
- net at D10.2 (A): now also D8.1 (K); no longer R4.1
- net at D11.2 (A): now also R3.1; no longer D9.1 (K)
- net at D7.1 (K): now also D9.2 (A); no longer R3.2
- new net: D3.1 (K), R1.2
- new net: D12.2 (A), R4.1
- new net: D9.1 (K), R3.2
Other:
- moved on the sheet: D10, D5, D9, R1, R3, R4
