File: Dayspring_Neo/Dayspring_Neo.kicad_pcb (KiCad board)
At the start: 2 copper layers, 310 x 11 mm, 36 parts, among them J1 IN, J2 OUT

Commit message: Production Version LED and 3030 Mounts
Parts:
- removed the G*** at (317.5, 33.4)
- added G***: LOGO, Daylight:RR_Logo_9mm_F-Silk, F.Cu at (317.5, 33.4)
Routing:
- net Net-(D12-Pad4): track 20.5 -> 22.3 mm
- net GND: vias 0 -> 57
Other:
- outline, holes or cut-outs redrawn
