File: Dayspring_Neo_Mini/Dayspring_Neo_Mini.kicad_sch (KiCad schematic)
At the start: 20 parts

Commit message: Production Version LED and 3030 Mounts
Parts:
- added C10, C11, C9: 0.1uF, Daylight:C_0805_2012Metric_Pad1.18x1.45mm_HandSolder_V3Dspec, symbol Device:C_Small
- added D10, D11, D9: LED_ALT, Daylight:XL-3528RGBW-WS2812B, symbol LED:SK6812
- C1, C2, C3, C4, C5, C6, C7, C8: value (none) -> 0.1uF; footprint (none) -> Daylight:C_0805_2012Metric_Pad1.18x1.45mm_HandSolder_V3Dspec
- D1, D2, D3, D4, D5, D6, D7, D8: value (none) -> LED_ALT; footprint (none) -> Daylight:XL-3528RGBW-WS2812B
- H1, H2: value (none) -> MountingHole; footprint (none) -> MountingHole:MountingHole_3.2mm_M3_Pad_Via
- J1: value (none) -> IN; footprint (none) -> Connector_JST:JST_XH_S3B-XH-A_1x03_P2.50mm_Horizontal
- J2: value (none) -> OUT; footprint (none) -> Connector_JST:JST_XH_S3B-XH-A_1x03_P2.50mm_Horizontal
Connections:
- net +5V: now also C10.1, C11.1, C9.1, D10.3 (VDD), D11.3 (VDD), D9.3 (VDD)
- net Dend: now also D11.4 (DOUT); no longer D8.4 (DOUT)
- net GND: now also C10.2, C11.2, C9.2, D10.1 (VSS), D11.1 (VSS), D9.1 (VSS)
- new net: D10.2 (DIN), D9.4 (DOUT)
- new net: D10.4 (DOUT), D11.2 (DIN)
- new net: D8.4 (DOUT), D9.2 (DIN)
Other:
- moved on the sheet: C1, C2, C3, C4, C5, C6, C7, C8, D1, D2, D3, D4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
